Commit message: diff_drive_control

File: src/diff_drive_description/models/xacro/base.xacro (robot description, xacro)
@@ -72,9 +72,9 @@
         </link>
         <!-- 调用轮子宏 -->
-        <xacro:wheel prefix="base_l" reflect="-1" />
-        <xacro:wheel prefix="base_r" reflect="1" />
+        <xacro:wheel prefix="left" reflect="1" />
+        <xacro:wheel prefix="right" reflect="-1" />
         <!-- 调用脚轮宏 -->
-        <xacro:caster prefix="front" reflect="-1" />
-        <xacro:caster prefix="back" reflect="1" />
+        <xacro:caster prefix="front" reflect="1" />
+        <xacro:caster prefix="back" reflect="-1" />
     </xacro:macro>
 </robot>

File: src/diff_drive_description/models/xacro/base_with_laser_camera.xacro (robot description, xacro)
@@ -1,7 +1,7 @@
 <?xml version="1.0"?>
 <robot name="mbot_with_laser_camera" xmlns:xacro="http://www.ros.org/wiki/xacro">
-    <xacro:include filename="$(find simulation_learning)/models/xacro/base.xacro" />
-    <xacro:include filename="$(find simulation_learning)/models/xacro/sensors/laser.xacro" />
-    <xacro:include filename="$(find simulation_learning)/models/xacro/sensors/camera.xacro" />
+    <xacro:include filename="$(find diff_drive_description)/models/xacro/base.xacro" />
+    <xacro:include filename="$(find diff_drive_description)/models/xacro/sensors/laser.xacro" />
+    <xacro:include filename="$(find diff_drive_description)/models/xacro/sensors/camera.xacro" />
     <xacro:property name="laser_offset_x" value="0" />
     <xacro:property name="laser_offset_y" value="0" />

File: src/diff_drive_description/models/xacro/gazebo/mbot_gazebo.xacro (robot description, xacro)
@@ -1,5 +1,5 @@
 <?xml version="1.0"?>
 <robot name="arm" xmlns:xacro="http://www.ros.org/wiki/xacro">
-    <xacro:include filename="$(find simulation_learning)/urdf/xacro/gazebo/mbot_base_gazebo.xacro" />
+    <xacro:include filename="$(find diff_drive_description)/urdf/xacro/gazebo/mbot_base_gazebo.xacro" />
     <mbot_base_gazebo/>
 </robot>

File: src/diff_drive_description/models/xacro/gazebo/mbot_with_camera_gazebo.xacro (robot description, xacro)
@@ -1,6 +1,6 @@
 <?xml version="1.0"?>
 <robot name="arm" xmlns:xacro="http://www.ros.org/wiki/xacro">
-    <xacro:include filename="$(find simulation_learning)/urdf/xacro/gazebo/mbot_base_gazebo.xacro" />
-    <xacro:include filename="$(find simulation_learning)/urdf/xacro/sensors/camera_gazebo.xacro" />
+    <xacro:include filename="$(find diff_drive_description)/urdf/xacro/gazebo/mbot_base_gazebo.xacro" />
+    <xacro:include filename="$(find diff_drive_description)/urdf/xacro/sensors/camera_gazebo.xacro" />
     <xacro:property name="camera_offset_x" value="0.17" />
     <xacro:property name="camera_offset_y" value="0" />

File: src/diff_drive_description/models/xacro/gazebo/mbot_with_kinect_gazebo.xacro (robot description, xacro)
@@ -1,6 +1,6 @@
 <?xml version="1.0"?>
 <robot name="arm" xmlns:xacro="http://www.ros.org/wiki/xacro">
-    <xacro:include filename="$(find simulation_learning)/urdf/xacro/gazebo/mbot_base_gazebo.xacro" />
-    <xacro:include filename="$(find simulation_learning)/urdf/xacro/sensors/kinect_gazebo.xacro" />
+    <xacro:include filename="$(find diff_drive_description)/urdf/xacro/gazebo/mbot_base_gazebo.xacro" />
+    <xacro:include filename="$(find diff_drive_description)/urdf/xacro/sensors/kinect_gazebo.xacro" />
     <xacro:property name="kinect_offset_x" value="0.15" />
     <xacro:property name="kinect_offset_y" value="0" />

File: src/diff_drive_description/models/xacro/gazebo/mbot_with_laser_gazebo.xacro (robot description, xacro)
@@ -1,6 +1,6 @@
 <?xml version="1.0"?>
 <robot name="arm" xmlns:xacro="http://www.ros.org/wiki/xacro">
-    <xacro:include filename="$(find simulation_learning)/urdf/xacro/gazebo/mbot_base_gazebo.xacro" />
-    <xacro:include filename="$(find simulation_learning)/urdf/xacro/sensors/lidar_gazebo.xacro" />
+    <xacro:include filename="$(find diff_drive_description)/urdf/xacro/gazebo/mbot_base_gazebo.xacro" />
+    <xacro:include filename="$(find diff_drive_description)/urdf/xacro/sensors/lidar_gazebo.xacro" />
     <xacro:property name="lidar_offset_x" value="0" />
     <xacro:property name="lidar_offset_y" value="0" />

File: src/diff_drive_description/models/xacro/mbot_base.xacro (robot description, xacro)
@@ -1,5 +1,5 @@
 <?xml version="1.0"?>
 <robot name="mbot_base" xmlns:xacro="http://www.ros.org/wiki/xacro">
-    <xacro:include filename="$(find simulation_learning)/models/xacro/base.xacro" />
+    <xacro:include filename="$(find diff_drive_description)/models/xacro/base.xacro" />
     <!-- 调用底盘宏 -->
     <xacro:mbot_base />

File: src/diff_drive_description/models/xacro/sensors/kinect.xacro (robot description, xacro)
@@ -7,5 +7,5 @@
                 <origin xyz="0 0 0" rpy="0 0 ${M_PI/2}"/>
                 <geometry>
-                    <mesh filename="package://simulation_learning/meshes/kinect.dae" />
+                    <mesh filename="package://diff_drive_description/meshes/kinect.dae" />
                 </geometry>
             </visual>

File: src/diff_drive_description/models/xacro/sensors/kinect_gazebo.xacro (robot description, xacro)
@@ -9,5 +9,5 @@
                 <origin xyz="0 0 0" rpy="0 0 ${M_PI/2}"/>
                 <geometry>
-                    <mesh filename="package://simulation_learning/meshes/kinect.dae" />
+                    <mesh filename="package://diff_drive_description/meshes/kinect.dae" />
                 </geometry>
             </visual>
