Commit message: 删除多余文件

File: src/diff_drive_description/models/base.xacro (robot description, xacro)
@@ -61,5 +61,5 @@
     </xacro:macro>
     <!-- 底盘宏定义 -->
-    <xacro:macro name="mbot_base">
+    <xacro:macro name="diff_drive_base">
         <link name="base_link">
             <visual>

File: src/diff_drive_description/models/diff_drive_robot.xacro (robot description, xacro)
@@ -1,7 +1,7 @@
 <?xml version="1.0"?>
-<robot name="mbot_with_laser_camera" xmlns:xacro="http://www.ros.org/wiki/xacro">
-    <xacro:include filename="$(find diff_drive_description)/models/xacro/base.xacro" />
-    <xacro:include filename="$(find diff_drive_description)/models/xacro/sensors/laser.xacro" />
-    <xacro:include filename="$(find diff_drive_description)/models/xacro/sensors/camera.xacro" />
+<robot name="diff_drive_robot" xmlns:xacro="http://www.ros.org/wiki/xacro">
+    <xacro:include filename="$(find diff_drive_description)/models/base.xacro" />
+    <xacro:include filename="$(find diff_drive_description)/models/sensors/laser.xacro" />
+    <xacro:include filename="$(find diff_drive_description)/models/sensors/camera.xacro" />
     <xacro:property name="laser_offset_x" value="0" />
     <xacro:property name="laser_offset_y" value="0" />
@@ -11,5 +11,5 @@
     <xacro:property name="camera_offset_z" value="0.165" />
     <!-- 调用base宏 -->
-    <xacro:mbot_base />
+    <xacro:diff_drive_base />
     <!-- laser_joint -->
     <joint name="laser_joint" type="fixed">
